Commit message: without prefix

File: robots/kobuki_hexagons_hokuyo.urdf.xacro (robot description, xacro)
@@ -1,6 +1,4 @@
 <?xml version="1.0"?>
 <robot name="turtlebot" xmlns:xacro="http://ros.org/wiki/xacro">
-<!-- Define prefix parameter with default value -->
-<xacro:property name="prefix" value="turtlebot/"/>
   <xacro:include filename="$(find turtlebot2_description)/urdf/turtlebot_common_library.urdf.xacro" />
   <xacro:include filename="$(find kobuki_description)/urdf/kobuki.urdf.xacro" />

File: robots/kobuki_hexagons_kinect.urdf.xacro (robot description, xacro)
@@ -1,6 +1,4 @@
 <?xml version="1.0"?>
 <robot name="turtlebot" xmlns:xacro="http://ros.org/wiki/xacro">
-<!-- Define prefix parameter with default value -->
-<xacro:property name="prefix" value="turtlebot/"/>
   <xacro:include filename="$(find turtlebot_description)/urdf/turtlebot_common_library.urdf.xacro" />
   <xacro:include filename="$(find kobuki_description)/urdf/kobuki.urdf.xacro" />

File: robots/kobuki_hexagons_kinect_hokuyo.urdf.xacro (robot description, xacro)
@@ -1,6 +1,4 @@
 <?xml version="1.0"?>
 <robot name="turtlebot" xmlns:xacro="http://www.ros.org/wiki/xacro">
-  <!-- Define prefix parameter with default value -->
-  <xacro:property name="prefix" value="turtlebot/"/>
   <xacro:include filename="$(find turtlebot2_description)/urdf/turtlebot_common_library.urdf.xacro"/>
   <xacro:include filename="$(find kobuki_description)/urdf/kobuki.urdf.xacro"/>

File: urdf/sensors/hokuyo.urdf.xacro (robot description, xacro)
@@ -16,10 +16,10 @@
     </material>
     <xacro:macro name="sensor_hokuyo" params="parent">
-        <joint name="${prefix}laser_joint" type="fixed">
+        <joint name="laser_joint" type="fixed">
             <origin xyz="${laser_px} ${laser_py} ${laser_pz}" rpy="0 0 0" />
             <parent link="${parent}" />
-            <child link="${prefix}laser" />
+            <child link="laser" />
         </joint>
-        <link name="${prefix}laser">
+        <link name="laser">
             <inertial>
                 <!-- change z into 0.025, this is the half of the box size -->

File: urdf/sensors/kinect.urdf.xacro (robot description, xacro)
@@ -6,22 +6,22 @@
   <!-- Parameterised in part by the values in turtlebot_properties.urdf.xacro -->
   <xacro:macro name="sensor_kinect" params="parent">
-    <joint name="${prefix}camera_rgb_joint" type="fixed">
+    <joint name="camera_rgb_joint" type="fixed">
       <origin xyz="${cam_px} ${kinect_cam_py} ${cam_pz}" rpy="${cam_or} ${cam_op} ${cam_oy}"/>
       <parent link="${parent}"/>
-      <child link="${prefix}camera_rgb_frame" />
+      <child link="camera_rgb_frame" />
     </joint>
-    <link name="${prefix}camera_rgb_frame"/>
-    <joint name="${prefix}camera_rgb_optical_joint" type="fixed">
+    <link name="camera_rgb_frame"/>
+    <joint name="camera_rgb_optical_joint" type="fixed">
       <origin xyz="0 0 0" rpy="${-M_PI/2} 0 ${-M_PI/2}" />
-      <parent link="${prefix}camera_rgb_frame" />
-      <child link="${prefix}camera_rgb_optical_frame" />
+      <parent link="camera_rgb_frame" />
+      <child link="camera_rgb_optical_frame" />
     </joint>
-    <link name="${prefix}camera_rgb_optical_frame"/>
-    <joint name="${prefix}camera_joint" type="fixed">
+    <link name="camera_rgb_optical_frame"/>
+    <joint name="camera_joint" type="fixed">
       <origin xyz="-0.031 ${-kinect_cam_py} -0.016" rpy="0 0 0"/>
-      <parent link="${prefix}camera_rgb_frame"/>
-      <child link="${prefix}camera_link"/>
+      <parent link="camera_rgb_frame"/>
+      <child link="camera_link"/>
     </joint>
-      <link name="${prefix}camera_link">
+      <link name="camera_link">
       <visual>
        <origin xyz="0 0 0" rpy="0 0 ${M_PI/2}"/>
@@ -47,16 +47,16 @@
          files. However, for Gazebo simulation we need them, so we add them here.
          (Hence, don't publish them additionally!) -->
-        <joint name="${prefix}camera_depth_joint" type="fixed">
+	<joint name="camera_depth_joint" type="fixed">
           <origin xyz="0 ${2 * -kinect_cam_py} 0" rpy="0 0 0" />
-          <parent link="${prefix}camera_rgb_frame" />
-          <child link="${prefix}camera_depth_frame" />
+	  <parent link="camera_rgb_frame" />
+	  <child link="camera_depth_frame" />
 	</joint>
-        <link name="${prefix}camera_depth_frame"/>
-        <joint name="${prefix}camera_depth_optical_joint" type="fixed">
+	<link name="camera_depth_frame"/>
+        <joint name="camera_depth_optical_joint" type="fixed">
           <origin xyz="0 0 0" rpy="${-M_PI/2} 0 ${-M_PI/2}" />
-          <parent link="${prefix}camera_depth_frame" />
-          <child link="${prefix}camera_depth_optical_frame" />
+	  <parent link="camera_depth_frame" />
+	  <child link="camera_depth_optical_frame" />
 	</joint>
-        <link name="${prefix}camera_depth_optical_frame"/>
+	<link name="camera_depth_optical_frame"/>
 	<!-- Kinect sensor for simulation -->
 	<xacro:turtlebot_sim_3dsensor/>

File: urdf/stacks/circles.urdf.xacro (robot description, xacro)
@@ -2,10 +2,10 @@
 <robot name="turtlebot_hardware" xmlns:xacro="http://ros.org/wiki/xacro">
   <xacro:macro name="turtlebot_spacer" params="parent number x_loc y_loc z_loc">
-    <joint name="${prefix}spacer_${number}_joint" type="fixed">
-      <origin xyz="${x_loc} ${y_loc} ${z_loc}" rpy="0 0 0" />
-      <parent link="${parent}"/>
-      <child link="${prefix}spacer_${number}_link" />
-    </joint>
-    <link name="${prefix}spacer_${number}_link">
+    <joint name="spacer_${number}_joint" type="fixed">
+      <origin xyz="${x_loc} ${y_loc} ${z_loc}" rpy="0 0 0" />
+      <parent link="${parent}"/>
+      <child link="spacer_${number}_link" />
+    </joint>
+    <link name="spacer_${number}_link">
       <inertial>
         <mass value="0.001" />
@@ -30,10 +30,10 @@
   </xacro:macro>
   <xacro:macro name="turtlebot_standoff_1in" params="parent number x_loc y_loc z_loc">
-    <joint name="${prefix}standoff_1in_${number}_joint" type="fixed">
-      <origin xyz="${x_loc} ${y_loc} ${z_loc}" rpy="0 0 0" />
-      <parent link="${parent}"/>
-      <child link="${prefix}standoff_1in_${number}_link" />
-    </joint>
-    <link name="${prefix}standoff_1in_${number}_link">
+    <joint name="standoff_1in_${number}_joint" type="fixed">
+      <origin xyz="${x_loc} ${y_loc} ${z_loc}" rpy="0 0 0" />
+      <parent link="${parent}"/>
+      <child link="standoff_1in_${number}_link" />
+    </joint>
+    <link name="standoff_1in_${number}_link">
       <inertial>
         <mass value="0.001" />
@@ -58,10 +58,10 @@
   </xacro:macro>
   <xacro:macro name="turtlebot_standoff_2in" params="parent number x_loc y_loc z_loc">
-    <joint name="${prefix}standoff_2in_${number}_joint" type="fixed">
-      <origin xyz="${x_loc} ${y_loc} ${z_loc}" rpy="0 0 0" />
-      <parent link="${parent}"/>
-      <child link="${prefix}standoff_2in_${number}_link" />
-    </joint>
-    <link name="${prefix}standoff_2in_${number}_link">
+    <joint name="standoff_2in_${number}_joint" type="fixed">
+      <origin xyz="${x_loc} ${y_loc} ${z_loc}" rpy="0 0 0" />
+      <parent link="${parent}"/>
+      <child link="standoff_2in_${number}_link" />
+    </joint>
+    <link name="standoff_2in_${number}_link">
       <inertial>
         <mass value="0.001" />
@@ -86,10 +86,10 @@
   </xacro:macro>
   <xacro:macro name="turtlebot_standoff_8in" params="parent number x_loc y_loc z_loc">
-    <joint name="${prefix}standoff_8in_${number}_joint" type="fixed">
-      <origin xyz="${x_loc} ${y_loc} ${z_loc}" rpy="0 0 0" />
-      <parent link="${parent}"/>
-      <child link="${prefix}standoff_8in_${number}_link" />
-    </joint>
-    <link name="${prefix}standoff_8in_${number}_link">
+    <joint name="standoff_8in_${number}_joint" type="fixed">
+      <origin xyz="${x_loc} ${y_loc} ${z_loc}" rpy="0 0 0" />
+      <parent link="${parent}"/>
+      <child link="standoff_8in_${number}_link" />
+    </joint>
+    <link name="standoff_8in_${number}_link">
       <inertial>
         <mass value="0.001" />
@@ -114,10 +114,10 @@
   </xacro:macro>
   <xacro:macro name="turtlebot_standoff_kinect" params="parent number x_loc y_loc z_loc">
-    <joint name="${prefix}standoff_kinect_${number}_joint" type="fixed">
-      <origin xyz="${x_loc} ${y_loc} ${z_loc}" rpy="0 0 0" />
-      <parent link="${parent}"/>
-      <child link="${prefix}standoff_kinect_${number}_link" />
-    </joint>
-    <link name="${prefix}standoff_kinect_${number}_link">
+    <joint name="standoff_kinect_${number}_joint" type="fixed">
+      <origin xyz="${x_loc} ${y_loc} ${z_loc}" rpy="0 0 0" />
+      <parent link="${parent}"/>
+      <child link="standoff_kinect_${number}_link" />
+    </joint>
+    <link name="standoff_kinect_${number}_link">
       <inertial>
         <mass value="0.001" />
@@ -146,10 +146,10 @@
     <xacro:turtlebot_spacer parent="${parent}" number="2" x_loc="-0.07239" y_loc="-0.1114679" z_loc="0.062992"/>
     <xacro:turtlebot_spacer parent="${parent}" number="3" x_loc="-0.07239" y_loc="0.1114679" z_loc="0.062992"/>
-    <joint name="${prefix}plate_0_joint" type="fixed">
+    <joint name="plate_0_joint" type="fixed">
       <origin xyz="-0.04334 0  0.06775704" rpy="0 0 0" />
       <parent link="${parent}"/>
-      <child link="${prefix}plate_0_link" />
-    </joint>
-    <link name="${prefix}plate_0_link">
+      <child link="plate_0_link" />
+    </joint>
+    <link name="plate_0_link">
       <inertial>
         <mass value="0.01" />
@@ -176,10 +176,10 @@
     <xacro:turtlebot_standoff_2in parent="${parent}" number="2" x_loc="-0.052832" y_loc="-0.1314196" z_loc="0.0709803"/>
     <xacro:turtlebot_standoff_2in parent="${parent}" number="3" x_loc="-0.052832" y_loc="0.1314196" z_loc="0.0709803"/>
-    <joint name="${prefix}plate_1_joint" type="fixed">
+    <joint name="plate_1_joint" type="fixed">
       <origin xyz="0.04068 0 0.05715" rpy="0 0 0" />
-      <parent link="${prefix}plate_0_link"/>
-      <child link="${prefix}plate_1_link" />
-    </joint>
-    <link name="${prefix}plate_1_link">
+      <parent link="plate_0_link"/>
+      <child link="plate_1_link" />
+    </joint>
+    <link name="plate_1_link">
       <inertial>
         <mass value="0.1" />
@@ -206,10 +206,10 @@
     <xacro:turtlebot_standoff_2in parent="standoff_2in_2_link" number="6" x_loc="0" y_loc="0" z_loc="0.05715"/>
     <xacro:turtlebot_standoff_2in parent="standoff_2in_3_link" number="7" x_loc="0" y_loc="0" z_loc="0.05715"/>
-    <joint name="${prefix}plate_2_joint" type="fixed">
+    <joint name="plate_2_joint" type="fixed">
       <origin xyz="0 0 0.0572008" rpy="0 0 0" />
-      <parent link="${prefix}plate_1_link"/>
-      <child link="${prefix}plate_2_link" />
-    </joint>
-    <link name="${prefix}plate_2_link">
+      <parent link="plate_1_link"/>
+      <child link="plate_2_link" />
+    </joint>
+    <link name="plate_2_link">
       <inertial>
         <mass value="0.01" />
@@ -238,10 +238,10 @@
     <xacro:turtlebot_standoff_8in parent="standoff_2in_6_link" number="2" x_loc="0" y_loc="0" z_loc="0.05715"/>
     <xacro:turtlebot_standoff_8in parent="standoff_2in_7_link" number="3" x_loc="0" y_loc="0" z_loc="0.05715"/>
-    <joint name="${prefix}plate_3_joint" type="fixed">
+    <joint name="plate_3_joint" type="fixed">
       <origin xyz="-0.01316 0 0.2063496" rpy="0 0 0" />
-      <parent link="${prefix}plate_2_link"/>
-      <child link="${prefix}plate_3_link" />
-    </joint>
-    <link name="${prefix}plate_3_link">
+      <parent link="plate_2_link"/>
+      <child link="plate_3_link" />
+    </joint>
+    <link name="plate_3_link">
       <inertial>
         <mass value="0.01" />

File: urdf/stacks/hexagons.urdf.xacro (robot description, xacro)
@@ -10,10 +10,10 @@
   <!-- Pole macros -->
   <xacro:macro name="stack_bottom_pole" params="parent number x_loc y_loc z_loc roll=0.0 pitch=0.0 yaw=0.0">
-    <joint name="${prefix}pole_bottom_${number}_joint" type="fixed">
+    <joint name="pole_bottom_${number}_joint" type="fixed">
       <origin xyz="${x_loc} ${y_loc} ${z_loc}" rpy="${roll} ${pitch} ${yaw}"/>
       <parent link="${parent}"/>
-      <child link="${prefix}pole_bottom_${number}_link"/>
-    </joint>
-    <link name="${prefix}pole_bottom_${number}_link">
+      <child link="pole_bottom_${number}_link"/>
+    </joint>
+    <link name="pole_bottom_${number}_link">
       <visual>
         <origin xyz="0 0 0" rpy="0 0 0"/>
@@ -38,10 +38,10 @@
   </xacro:macro>
   <xacro:macro name="stack_middle_pole" params="parent number x_loc y_loc z_loc roll=0.0 pitch=0.0 yaw=0.0">
-    <joint name="${prefix}pole_middle_${number}_joint" type="fixed">
+    <joint name="pole_middle_${number}_joint" type="fixed">
       <origin xyz="${x_loc} ${y_loc} ${z_loc}" rpy="${roll} ${pitch} ${yaw}" />
       <parent link="${parent}"/>
-      <child link="${prefix}pole_middle_${number}_link"/>
-    </joint>
-    <link name="${prefix}pole_middle_${number}_link">
+      <child link="pole_middle_${number}_link"/>
+    </joint>
+    <link name="pole_middle_${number}_link">
       <visual>
         <origin xyz="0 0 0" rpy="0 ${M_PI} 0"/>
@@ -66,10 +66,10 @@
   </xacro:macro>
   <xacro:macro name="stack_top_pole" params="parent number x_loc y_loc z_loc roll=0.0 pitch=0.0 yaw=0.0">
-    <joint name="${prefix}pole_top_${number}_joint" type="fixed">
+    <joint name="pole_top_${number}_joint" type="fixed">
       <origin xyz="${x_loc} ${y_loc} ${z_loc}" rpy="${roll} ${pitch} ${yaw}"/>
       <parent link="${parent}"/>
-      <child link="${prefix}pole_top_${number}_link"/>
-    </joint>
-    <link name="${prefix}pole_top_${number}_link">
+      <child link="pole_top_${number}_link"/>
+    </joint>
+    <link name="pole_top_${number}_link">
       <visual>
         <origin xyz=" 0 0 0" rpy="0 0 0"/>
@@ -94,10 +94,10 @@
   </xacro:macro>
   <xacro:macro name="stack_3d_sensor_pole" params="parent number x_loc y_loc z_loc roll=0.0 pitch=0.0 yaw=0.0">
-    <joint name="${prefix}pole_kinect_${number}_joint" type="fixed">
+    <joint name="pole_kinect_${number}_joint" type="fixed">
       <origin xyz="${x_loc} ${y_loc} ${z_loc}" rpy="${roll} ${pitch} ${yaw}"/>
       <parent link="${parent}"/>
-      <child link="${prefix}pole_kinect_${number}_link"/>
-    </joint>
-    <link name="${prefix}pole_kinect_${number}_link">
+      <child link="pole_kinect_${number}_link"/>
+    </joint>
+    <link name="pole_kinect_${number}_link">
       <visual>
         <origin xyz="0 0 0" rpy="0 0 0"/>
@@ -133,10 +133,10 @@
     <xacro:stack_bottom_pole parent="${parent}" number="4" x_loc= "0.055" y_loc="-0.120" z_loc="0.1028"/>
     <xacro:stack_bottom_pole parent="${parent}" number="5" x_loc="-0.055" y_loc="-0.120" z_loc="0.1028"/>
-    <joint name="${prefix}plate_bottom_joint" type="fixed">
+    <joint name="plate_bottom_joint" type="fixed">
       <origin xyz="0.02364 0.0 0.1306" rpy="0 0 0"/>
       <parent link="${parent}"/>
-      <child link="${prefix}plate_bottom_link"/>
-    </joint>
-    <link name="${prefix}plate_bottom_link">
+      <child link="plate_bottom_link"/>
+    </joint>
+    <link name="plate_bottom_link">
       <visual>
         <origin xyz="0 0 0" rpy="0 0 0"/>
@@ -163,10 +163,10 @@
     <xacro:stack_middle_pole parent="${parent}" number="2" x_loc="-0.0381" y_loc= "0.1505" z_loc="0.1640"/>
     <xacro:stack_middle_pole parent="${parent}" number="3" x_loc="-0.0381" y_loc="-0.1505" z_loc="0.1640"/>
-    <joint name="${prefix}plate_middle_joint" type="fixed">
+    <joint name="plate_middle_joint" type="fixed">
       <origin xyz="-0.01364 0.0 0.1874" rpy="0 0 0"/>
       <parent link="${parent}"/>
-      <child link="${prefix}plate_middle_link"/>
-    </joint>
-    <link name="${prefix}plate_middle_link">
+      <child link="plate_middle_link"/>
+    </joint>
+    <link name="plate_middle_link">
       <visual>
         <origin xyz="0 0 0" rpy="0 0 0"/>
@@ -197,10 +197,10 @@
     <xacro:stack_3d_sensor_pole parent="${parent}" number="0" x_loc="0.1024" y_loc= "0.098" z_loc="0.2372"/>
     <xacro:stack_3d_sensor_pole parent="${parent}" number="1" x_loc="0.1024" y_loc="-0.098" z_loc="0.2372"/>
-    <joint name="${prefix}plate_top_joint" type="fixed">
+    <joint name="plate_top_joint" type="fixed">
       <origin xyz="-0.01364 0.0  0.3966" rpy="0 0 0"/>
       <parent link="${parent}"/>
-      <child link="${prefix}plate_top_link"/>
-    </joint>
-    <link name="${prefix}plate_top_link">
+      <child link="plate_top_link"/>
+    </joint>
+    <link name="plate_top_link">
       <visual>
         <origin xyz="0 0 0" rpy="0 0 0"/>
